File: emoc.kicad_pcb (KiCad board)
At the start: 4 copper layers, 42 parts, among them J1 XT60PW-M, Q1 NVMFS5C604NL, Q2 NVMFS5C604NL, Q3 NVMFS5C604NL, Q4 NVMFS5C604NL, Q5 NVMFS5C604NL, Q6 NVMFS5C604NL, U1 STM32F303CBTx, U2 DRV8323R

Commit message: still work in progress
Parts:
- added 10k1: R_US, Resistor_SMD:R_0603_1608Metric, F.Cu at (131.6, 113.0)
- added 10k2: R_US, Resistor_SMD:R_0603_1608Metric, F.Cu at (84.0, 95.6)
- added C26: 1u, Capacitor_SMD:C_0805_2012Metric, F.Cu at (120.8, 86.5)
- added C27: 10n, Capacitor_SMD:C_0603_1608Metric, F.Cu at (120.6, 89.3)
- added C28: 100n, Capacitor_SMD:C_0603_1608Metric, F.Cu at (142.5, 91.1)
- added C29: 100n, Capacitor_SMD:C_0603_1608Metric, F.Cu at (127.8, 91.4)
- added C30: 100n, Capacitor_SMD:C_0603_1608Metric, F.Cu at (126.9, 84.1)
- added C31: 100n, Capacitor_SMD:C_0603_1608Metric, F.Cu at (108.3, 84.4)
- added C32: 100n, Capacitor_SMD:C_0603_1608Metric, F.Cu at (111.7, 90.0)
- added C33: 100n, Capacitor_SMD:C_0603_1608Metric, F.Cu at (111.7, 86.0)
- added C34: 1u, Capacitor_SMD:C_1206_3216Metric, F.Cu at (108.7, 89.2)
- added C35: 100n, Capacitor_SMD:C_0603_1608Metric, F.Cu at (100.2, 83.9)
- added C36: 100n, Capacitor_SMD:C_0603_1608Metric, F.Cu at (101.0, 73.9)
- added C37: 220p, Capacitor_SMD:C_0603_1608Metric, F.Cu at (131.6, 115.5)
- added C38: 220p, Capacitor_SMD:C_0603_1608Metric, F.Cu at (126.4, 119.7)
- added C4: TBD, Capacitor_SMD:C_0603_1608Metric, F.Cu at (195.2, 114.6)
- added C5: TBD, Capacitor_SMD:C_0603_1608Metric, F.Cu at (195.2, 117.1)
- added C6: TBD, Capacitor_SMD:C_0603_1608Metric, F.Cu at (199.2, 114.6)
- added C9: 100n, Capacitor_SMD:C_0603_1608Metric, B.Cu at (144.5, 95.3)
- added H1: MountingHole_Pad, MountingHole:MountingHole_3.2mm_M3_Pad, F.Cu at (186.0, 96.0)
- added H2: MountingHole_Pad, MountingHole:MountingHole_3.2mm_M3_Pad, F.Cu at (114.0, 96.0)
- added J2: RJHSE-x38x-02_CAN, libysk_Connector_Jack:RJHSE-x38x-02, F.Cu at (116.0, 75.8)
- added J3: Conn_01x04, libysk_Connector_TE:EP25_1744426-4, F.Cu at (157.0, 50.1)
- added L2: L, Inductor_SMD:L_1210_3225Metric, F.Cu at (116.6, 71.8)
- added NT1: Net-Tie_2, NetTie:NetTie-2_SMD_Pad0.5mm, F.Cu at (174.1, 104.0)
- added Q7: BSS138, Package_TO_SOT_SMD:SOT-23, F.Cu at (80.6, 99.4)
- added R19: 10k, Resistor_SMD:R_0603_1608Metric, F.Cu at (132.1, 96.3)
- added R20: R_US, Resistor_SMD:R_0603_1608Metric, F.Cu at (118.5, 71.0)
- added R21: R_US, Resistor_SMD:R_0603_1608Metric, F.Cu at (118.5, 73.5)
- added R22: 100R, Resistor_SMD:R_0603_1608Metric, F.Cu at (76.0, 97.1)
- added R23: 51k1, Resistor_SMD:R_0603_1608Metric, F.Cu at (130.4, 118.0)
- added R24: 100R, Resistor_SMD:R_0603_1608Metric, F.Cu at (135.6, 115.5)
- added R25: 100R, Resistor_SMD:R_0603_1608Metric, F.Cu at (130.4, 120.5)
- added TP1: TestPoint, TestPoint:TestPoint_Pad_D1.0mm, B.Cu at (172.1, 73.2)
- added TP2: TestPoint, TestPoint:TestPoint_Pad_D1.0mm, B.Cu at (162.1, 74.0)
- added TP3: TestPoint, TestPoint:TestPoint_Pad_D1.0mm, B.Cu at (194.9, 101.2)
- added TP4: TestPoint, TestPoint:TestPoint_Pad_D1.0mm, B.Cu at (194.4, 99.3)
- added TP5: TestPoint, TestPoint:TestPoint_Pad_D1.0mm, B.Cu at (172.5, 90.0)
- added TP6: TestPoint, TestPoint:TestPoint_Pad_D1.0mm, B.Cu at (162.6, 90.8)
- added U3: MC78L05_SOT89, Package_TO_SOT_SMD:SOT-89-3, B.Cu at (108.0, 61.0)
- added U4: TPS562201, Package_TO_SOT_SMD:SOT-23-6, F.Cu at (104.3, 72.0)
- added U5: Si8621AB-B-IS, Package_SO:SOIC-8_3.9x4.9mm_P1.27mm, F.Cu at (110.3, 104.4)
- added U6: NCV7351D13, Package_SO:SOIC-8_3.9x4.9mm_P1.27mm, F.Cu at (110.3, 96.3)
- added U7: TLP291, Package_SO:SOIC-4_4.55x2.6mm_P1.27mm, F.Cu at (92.5, 97.0)
- C7: moved to B.Cu
- moved U1 38.5 mm to (135.3, 87.8), turned to 45 degrees
- moved R11 26.2 mm to (153.1, 96.9)
- moved R12 26.2 mm to (149.4, 96.4)
- moved R8 23.3 mm to (142.5, 70.8)
- moved R10 21.1 mm to (141.4, 98.2)
- moved R9 19.1 mm to (139.0, 71.0)
- moved R6 7.44 mm to (149.0, 71.7)
- moved R7 6.93 mm to (148.7, 75.6)
- moved R17 4.47 mm to (172.8, 88.5)
- moved C25 4.32 mm to (177.7, 88.5)
- moved C23 4.30 mm to (169.1, 88.5)
- moved C24 4.30 mm to (165.6, 88.5)
- moved R13 4.19 mm to (173.1, 96.9)
- moved C17 4.19 mm to (169.3, 96.9)
- moved C7 4.19 mm to (145.8, 79.8), turned to 180 degrees
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Connections:
- net Net-(Q2-Pad1) renamed /emoc_page3/SL_A
- net Net-(Q6-Pad1) renamed /emoc_page3/SL_C
- Q4 pad 1: Net-(Q4-Pad1) -> /emoc_page3/SL_B
- Q4 pad 2: Net-(Q4-Pad1) -> /emoc_page3/SL_B
- Q4 pad 3: Net-(Q4-Pad1) -> /emoc_page3/SL_B
- R18 pad 1: Net-(Q4-Pad1) -> /emoc_page3/SL_B
- R2 pad 1: GND -> /emoc_page3/SL_B
- R2 pad 2: SN_B -> SP_B
- R2 pad 3: SP_B -> SN_B
- R2 pad 4: Net-(Q4-Pad1) -> GND
- U1 pad 1: Net-(U1-Pad1) -> +3V3
- U1 pad 14: Net-(U1-Pad14) -> ~SS
- U1 pad 15: Net-(U1-Pad15) -> SCK
- U1 pad 16: Net-(U1-Pad16) -> MISO
- U1 pad 17: Net-(U1-Pad17) -> MOSI
- U1 pad 23: Net-(U1-Pad23) -> GND
- U1 pad 24: Net-(U1-Pad24) -> +3V3
- U1 pad 26: Net-(U1-Pad26) -> INL_A
- U1 pad 27: Net-(U1-Pad27) -> INL_B
- U1 pad 28: Net-(U1-Pad28) -> INL_C
- U1 pad 29: Net-(U1-Pad29) -> INH_A
- U1 pad 30: Net-(U1-Pad30) -> INH_B
- U1 pad 31: Net-(U1-Pad31) -> INH_C
- U1 pad 35: Net-(U1-Pad35) -> GND
- U1 pad 36: Net-(U1-Pad36) -> +3V3
- U1 pad 45: Net-(U1-Pad45) -> CAN_RX
- U1 pad 46: Net-(U1-Pad46) -> CAN_TX
- U1 pad 47: Net-(U1-Pad47) -> GND
- U1 pad 48: Net-(U1-Pad48) -> +3V3
- U2 pad 26: Net-(C9-Pad1) -> VDDA
- U2 pad 29: SDO -> MISO
- U2 pad 30: SDI -> MOSI
- U2 pad 31: SCLK -> SCK
- U2 pad 32: SCS -> ~SS
Routing:
- net SP_B: track 0.00 -> 11.3 mm, vias 0 -> 2
- net GL_B: track 5.09 -> 16.1 mm, vias 1 -> 2
- net SP_C: track 0.00 -> 10.5 mm
- net SN_B: track 0.00 -> 10.0 mm, vias 0 -> 2
- net SN_A: track 8.69 -> 17.6 mm, vias 0 -> 2
- net INH_C: track 0.00 -> 8.65 mm, vias 0 -> 1
- net ~SS: track 0.00 -> 8.02 mm, vias 0 -> 1
- net SCK: track 0.00 -> 7.62 mm, vias 0 -> 1
- net SP_A: track 11.7 -> 19.1 mm, vias 0 -> 2
- net INL_C: track 0.00 -> 7.28 mm, vias 0 -> 1
- net MISO: track 0.00 -> 6.67 mm, vias 0 -> 1
- net MOSI: track 0.00 -> 6.19 mm, vias 0 -> 1
- net INH_A: track 0.00 -> 5.69 mm, vias 0 -> 1
- net INH_B: track 0.00 -> 5.48 mm, vias 0 -> 1
- net GL_C: track 18.1 -> 12.7 mm
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- added copper zone on B.Cu, net /emoc_page3/SL_A
- added copper zone on B.Cu, net /emoc_page3/SL_B
- added copper zone on B.Cu, net /emoc_page3/SL_C
- added copper zone on B.Cu, net GND
- added copper zone on F.Cu, net GND
- added copper zone on B.Cu, net GNDD
- added copper zone on B.Cu, net SH_A
- added copper zone on B.Cu, net SH_B
- added copper zone on B.Cu, net SH_C
- added copper zone on B.Cu, net VDC
Other:
- board outline added: 80 x 50 mm
- net class Default: via_dia 0.8 -> 0.5; via_drill 0.4 -> 0.2
- rule via_min_drill: 0.3 -> 0.2

Commit message: idk
Parts:
- added C14: 100n, Capacitor_SMD:C_0603_1608Metric, F.Cu at (143.0, 88.0)
- moved C4 61.5 mm to (136.0, 98.0)
- moved R25 60.9 mm to (153.0, 64.0), turned to 90 degrees
- moved C38 59.0 mm to (153.0, 67.0)
- moved C37 57.0 mm to (158.0, 65.0)
- moved R24 55.0 mm to (155.0, 64.0), turned to 90 degrees
- moved R6 16.7 mm to (134.0, 79.0), turned to 270 degrees
