File: emoc_page2.sch (KiCad schematic (older format))
At the start: 1 part, among them U1 STM32F303CBTx

Commit message: still work in progress
Parts:
- added C26: 1u, Capacitor_SMD:C_0805_2012Metric, symbol Device:C_Small
- added C27: 10n, Capacitor_SMD:C_0603_1608Metric, symbol Device:C_Small
- added C28, C29, C30: 100n, Capacitor_SMD:C_0603_1608Metric, symbol Device:C_Small
- added FB1: Ferrite_Bead_Small, symbol Device:Ferrite_Bead_Small
- added R19: 10k, Resistor_SMD:R_0603_1608Metric, symbol Device:R_US
Connections:
- net +3V3: now reaches U1.1 (VBAT)
- net +3V3: now also U1.24 (VDD), U1.36 (VDD), U1.48 (VDD), C28.1, C29.1, C30.1, FB1.1, R19.2
- net ~SS: now reaches U1.14 (PA4)
- net SCK: now reaches U1.15 (PA5)
- net MISO: now reaches U1.16 (PA6)
- net MOSI: now reaches U1.17 (PA7)
- net GND: now reaches U1.23 (VSS)
- net GND: now also U1.35 (VSS), U1.47 (VSS), C26.2, C27.2, C28.2, C29.2, C30.2
- net INL_A: now reaches U1.26 (PB13)
- net INL_B: now reaches U1.27 (PB14)
- net INL_C: now reaches U1.28 (PB15)
- net INH_A: now reaches U1.29 (PA8)
- net INH_B: now reaches U1.30 (PA9)
- net INH_C: now reaches U1.31 (PA10)
- net CAN_RX: now reaches U1.45 (PB8)
- net CAN_TX: now reaches U1.46 (PB9)
- net at U1.7 (NRST): now also R19.1
- net at U1.9 (VDDA): now also C26.1, C27.1, FB1.2

Commit message: idk
Connections:
- wire segments 43 -> 46
Changed lines of the file:
@@
 Wire Wire Line
 	4350 4150 4550 4150
+Wire Wire Line
+	4350 3450 4550 3450
+Wire Wire Line
+	3050 3550 2850 3550
+Wire Wire Line
+	3050 3650 2850 3650
 $EndSCHEMATC
